Commit message: modified

File: urdfs/robot_hand_finger1.urdf (robot description, URDF)
Before this commit: robot pi_robot, 3 links, 1 joints
Links:
- removed link finger1
- removed link finger2
- removed link finger3
- added link finger1_1; visual box size=0.02 0.02 0.045
- added link finger1_2; visual box size=0.02 0.02 0.025
- added link finger1_3; visual box size=0.02 0.02 0.02
Joints:
- removed joint forearm_palm_joint
- added joint finger1_1_finger1_2_joint: type revolute, parent finger1_1, child finger1_2, origin xyz=0 0 0.045 rpy=0 0 0, axis 0 1 0, limit lower=-3.1416 upper=3.1416 effort=10 velocity=3
- added joint finger1_2_finger1_3_joint: type revolute, parent finger1_2, child finger1_3, origin xyz=0 0 0.02 rpy=0 0 0, axis 0 1 0, limit lower=-3.1416 upper=3.1416 effort=10 velocity=3

File: urdfs/robot_hand_finger2.urdf (robot description, URDF)
Before this commit: robot pi_robot, 3 links, 1 joints
Links:
- removed link finger1
- removed link finger2
- removed link finger3
- added link finger2_1; visual box size=0.02 0.02 0.05
- added link finger2_2; visual box size=0.02 0.02 0.03
- added link finger2_3; visual box size=0.02 0.02 0.02
Joints:
- removed joint forearm_palm_joint
- added joint finger1_2_finger1_3_joint: type revolute, parent finger2_2, child finger2_3, origin xyz=0 0 0.03 rpy=0 0 0, axis 0 1 0, limit lower=-3.1416 upper=3.1416 effort=10 velocity=3
- added joint finger2_1_finger2_2_joint: type revolute, parent finger2_1, child finger2_2, origin xyz=0 0 0.05 rpy=0 0 0, axis 0 1 0, limit lower=-3.1416 upper=3.1416 effort=10 velocity=3

File: urdfs/robot_hand_finger3.urdf (robot description, URDF)
Before this commit: robot pi_robot, 3 links, 1 joints
Links:
- removed link finger1
- removed link finger2
- removed link finger3
- added link finger3_1; visual box size=0.02 0.02 0.045
- added link finger3_2; visual box size=0.02 0.02 0.025
- added link finger3_3; visual box size=0.02 0.02 0.02
Joints:
- removed joint forearm_palm_joint
- added joint finger3_1_finger2_2_joint: type revolute, parent finger3_1, child finger3_2, origin xyz=0 0 0.045 rpy=0 0 0, axis 0 1 0, limit lower=-3.1416 upper=3.1416 effort=10 velocity=3
- added joint finger3_2_finger2_3_joint: type revolute, parent finger3_2, child finger3_3, origin xyz=0 0 0.02 rpy=0 0 0, axis 0 1 0, limit lower=-3.1416 upper=3.1416 effort=10 velocity=3

File: urdfs/robot_hand_finger4.urdf (robot description, URDF)
Before this commit: robot pi_robot, 3 links, 1 joints
Links:
- removed link finger1
- removed link finger2
- removed link finger3
- added link finger4_1; visual box size=0.02 0.02 0.035
- added link finger4_2; visual box size=0.02 0.02 0.02
- added link finger4_3; visual box size=0.02 0.02 0.02
Joints:
- removed joint forearm_palm_joint
- added joint finger4_1_finger4_2_joint: type revolute, parent finger4_1, child finger4_2, origin xyz=0 0 0.035 rpy=0 0 0, axis 0 1 0, limit lower=-3.1416 upper=3.1416 effort=10 velocity=3
- added joint finger4_2_finger4_3_joint: type revolute, parent finger4_2, child finger4_3, origin xyz=0 0 0.02 rpy=0 0 0, axis 0 1 0, limit lower=-3.1416 upper=3.1416 effort=10 velocity=3
